File: Projects/Power Tower Mast/m/n.sch (EAGLE design)
At the start: 42 parts

Commit message: final updates before fab.  added new letters for future projects.
Parts:
- removed LED22, LED23, LED24: (no value), CyberRailGuru:LED0805
- removed VO15, VO16, VO8, VO9: (no value), CyberRailGuru:TEST_POINTPAD1-20
- added VO08, VO09: (no value), CyberRailGuru:TEST_POINTPAD1-20
Connections:
- removed net N$1 (its old number): LED23.C, LED24.A
- removed net N$2 (its old number): LED22.C, LED23.A
- removed net VOUT8: LED24.C, VO16.TP, VO8.TP
- net VIN: no longer LED22.A
- net VOUT1: now also VO08.TP; no longer VO9.TP
- net VOUT2: now also VO09.TP; no longer VO10.TP
- net VOUT3: now also VO10.TP; no longer VO11.TP
- net VOUT4: now also VO11.TP; no longer VO12.TP
- net VOUT5: now also VO12.TP; no longer VO13.TP
- net VOUT6: now also VO13.TP; no longer VO14.TP
- net VOUT7: now also VO14.TP; no longer VO15.TP
Other:
- moved on the sheet: LED1, LED10, LED11, LED12, LED13, LED14, LED15, LED16, LED17, LED18, LED19, LED2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
