File: Projects/Power Tower Mast/o/i.brd (EAGLE design)
At the start: 16.5 x 21.6 mm, 27 parts

Commit message: final updates before fab.  added new letters for future projects.
Parts:
- moved VO3 8.49 mm to (9.37, 12.1)
- moved LED10 7.79 mm to (8.26, 14.9), turned to 270 degrees
- moved LED4 6.83 mm to (4.76, 2.22), turned to 0 degrees
- moved VO8 6.74 mm to (9.37, 13.7)
- moved LED9 6.35 mm to (8.26, 12.9), turned to 270 degrees
- moved VO2 6.19 mm to (9.37, 6.03)
- moved VO7 6.19 mm to (9.37, 7.62)
- moved LED8 6.19 mm to (8.26, 10.8), turned to 270 degrees
- moved LED7 5.87 mm to (8.26, 8.89), turned to 270 degrees
- moved LED6 5.71 mm to (8.26, 6.83), turned to 270 degrees
- moved LED5 5.56 mm to (8.26, 4.76), turned to 270 degrees
- moved LED11 5.18 mm to (8.26, 16.8), turned to 270 degrees
- moved LED3 3.82 mm to (7.14, 2.22), turned to 0 degrees
- moved LED13 3.65 mm to (7.14, 19.4), turned to 0 degrees
- moved LED1 3.58 mm to (11.7, 2.22), turned to 0 degrees
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Connections:
- removed net N$1: LED13.A, LED14.C
- removed net N$2: LED14.A, LED15.C
- new net N$19: LED14.C, LED15.A
- new net N$20: LED13.C, LED14.A
- net VIN: now also LED13.A; no longer LED15.A
- net VOUT5: now also LED15.C; no longer LED13.C
Routing:
- net N$15: track 2.89 -> 8.47 mm, vias 0 -> 2
- net VIN: track 35.1 -> 30.1 mm
- net N$19: track 0.00 -> 3.25 mm
- net N$20: track 0.00 -> 3.09 mm
- net N$2: track 2.89 -> 0.00 mm
- net N$1: track 2.89 -> 0.00 mm
- net VOUT2: track 2.60 -> 1.64 mm
Other:
- board text added: "I"
- board text removed: "T"
