File: Projects/Power Tower Mast/o/i.sch (EAGLE design)
At the start: 42 parts

Commit message: final updates before fab.  added new letters for future projects.
Parts:
- removed LED16, LED17, LED18, LED19, LED20, LED21, LED22, LED23, LED24: (no value), CyberRailGuru:LED0805
- removed VO11, VO12, VO13, VO14, VO15, VO16: (no value), CyberRailGuru:TEST_POINTPAD1-20
Connections:
- removed net N$1: LED23.C, LED24.A
- removed net N$2: LED22.C, LED23.A
- removed net N$61: LED17.C, LED18.A
- removed net N$62: LED16.C, LED17.A
- removed net N$63: LED20.C, LED21.A
- removed net N$64: LED19.C, LED20.A
- removed net VOUT6: LED18.C, VO14.TP, VO6.TP
- removed net VOUT7: LED21.C, VO15.TP, VO7.TP
- removed net VOUT8: LED24.C, VO16.TP, VO8.TP
- net VIN: no longer LED16.A, LED19.A, LED22.A
- net VOUT1: now also VO6.TP; no longer VO9.TP
- net VOUT2: now also VO7.TP; no longer VO10.TP
- net VOUT3: now also VO8.TP; no longer VO11.TP
- net VOUT4: now also VO9.TP; no longer VO12.TP
- net VOUT5: now also VO10.TP; no longer VO13.TP
Other:
- moved on the sheet: LED1, LED10, LED11, LED12, LED13, LED14, LED15, LED2, LED3, LED4, LED5, LED6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
