File: Projects/Power Tower Mast/o/u.brd (EAGLE design)
At the start: 16.5 x 21.6 mm, 27 parts

Commit message: final updates before fab.  added new letters for future projects.
Parts:
- added LED16, LED17, LED18, LED19, LED20, LED21: (no value), CyberRailGuru:LED_0805
- added VO11, VO12, VO13, VO14: (no value), CyberRailGuru:P1-20
- moved VO8 14.1 mm to (3.17, 6.83)
- moved LED10 12.2 mm to (14.0, 20.0), turned to 90 degrees
- moved VO7 10.9 mm to (5.40, 2.54)
- moved LED11 10.4 mm to (14.0, 17.9), turned to 90 degrees
- moved LED15 9.55 mm to (14.0, 9.68), turned to 90 degrees
- moved LED12 9.05 mm to (14.0, 15.9), turned to 90 degrees
- moved VO5 8.70 mm to (12.9, 8.89)
- moved VO10 8.53 mm to (3.65, 20.8)
- moved VO4 7.96 mm to (12.9, 16.7)
- moved LED14 7.57 mm to (14.0, 11.7), turned to 90 degrees
- moved VIN 6.74 mm to (2.86, 2.54)
- moved LED13 6.26 mm to (14.0, 13.8), turned to 90 degrees
- moved LED3 5.98 mm to (2.54, 7.62), turned to 270 degrees
- moved LED4 5.93 mm to (2.54, 9.68), turned to 270 degrees
- moved LED5 5.89 mm to (2.54, 11.7), turned to 270 degrees
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Connections:
- removed net N$1: LED13.A, LED14.C
- removed net N$2: LED14.A, LED15.C
- new net N$19: LED14.C, LED15.A
- new net N$20: LED13.C, LED14.A
- new net N$23: LED17.C, LED18.A
- new net N$24: LED16.C, LED17.A
- new net N$27: LED20.C, LED21.A
- new net N$28: LED19.C, LED20.A
- new net VOUT6: LED18.C, VO13.TP, VO6.TP
- new net VOUT7: LED21.C, VO14.TP, VO7.TP
- net VIN: now also LED13.A, LED16.A, LED19.A; no longer LED15.A
- net VOUT1: now also VO8.TP; no longer VO6.TP
- net VOUT2: now also VO9.TP; no longer VO7.TP
- net VOUT3: now also VO10.TP; no longer VO8.TP
- net VOUT4: now also VO11.TP; no longer VO9.TP
- net VOUT5: now also LED15.C, VO12.TP; no longer LED13.C, VO10.TP
Routing:
- net VIN: track 35.1 -> 47.7 mm, vias 4 -> 6
- net N$24: track 0.00 -> 3.96 mm
- net N$23: track 0.00 -> 3.94 mm
- net N$19: track 0.00 -> 2.95 mm
- net N$27: track 0.00 -> 2.95 mm
- net N$20: track 0.00 -> 2.95 mm
- net N$28: track 0.00 -> 2.95 mm
- net N$2: track 2.89 -> 0.00 mm
- net N$1: track 2.89 -> 0.00 mm
- net VOUT6: track 0.00 -> 2.20 mm
- net VOUT7: track 0.00 -> 1.92 mm
- net VOUT2: track 2.60 -> 1.64 mm
Other:
- board text added: "U"
- board text removed: "T"
