File: Projects/Power Tower Mast/p/p.sch (EAGLE design)
At the start: 25 parts

Commit message: updated with extra vias and panelized
Parts:
- added VIN1, VO10, VO11, VO12, VO7, VO8, VO9: (no value), CyberRailGuru:TEST_POINTPAD1-20
Connections:
- net VIN: now also VIN1.TP
- net VOUT1: now also VO7.TP
- net VOUT2: now also VO8.TP
- net VOUT3: now also VO9.TP
- net VOUT4: now also VO10.TP
- net VOUT5: now also VO11.TP
- net VOUT6: now also VO12.TP
Changed lines of the file:
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@@
 <part name="VO6" library="CyberRailGuru" deviceset="TEST_POINT" device="PAD1-20"/>
 <part name="FRAME1" library="SparkFun-Aesthetics" deviceset="FRAME-A3" device=""/>
+<part name="VIN1" library="CyberRailGuru" deviceset="TEST_POINT" device="PAD1-20"/>
+<part name="VO7" library="CyberRailGuru" deviceset="TEST_POINT" device="PAD1-20"/>
+<part name="VO8" library="CyberRailGuru" deviceset="TEST_POINT" device="PAD1-20"/>
+<part name="VO9" library="CyberRailGuru" deviceset="TEST_POINT" device="PAD1-20"/>
+<part name="VO10" library="CyberRailGuru" deviceset="TEST_POINT" device="PAD1-20"/>
+<part name="VO11" library="CyberRailGuru" deviceset="TEST_POINT" device="PAD1-20"/>
+<part name="VO12" library="CyberRailGuru" deviceset="TEST_POINT" device="PAD1-20"/>
 </parts>
 <sheets>
@@
 <instance part="LED17" gate="G$1" x="50.8" y="187.96" rot="R90"/>
 <instance part="LED16" gate="G$1" x="40.64" y="187.96" rot="R90"/>
-<instance part="VIN" gate="G$1" x="27.94" y="180.34" rot="R180"/>
-<instance part="VO1" gate="G$1" x="76.2" y="238.76" rot="R270"/>
-<instance part="VO2" gate="G$1" x="76.2" y="228.6" rot="R270"/>
-<instance part="VO3" gate="G$1" x="76.2" y="218.44" rot="R270"/>
-<instance part="VO4" gate="G$1" x="76.2" y="208.28" rot="R270"/>
-<instance part="VO5" gate="G$1" x="76.2" y="198.12" rot="R270"/>
-<instance part="VO6" gate="G$1" x="76.2" y="187.96" rot="R270"/>
+<instance part="VIN" gate="G$1" x="27.94" y="180.34" smashed="yes" rot="R180">
+<attribute name="NAME" x="29.21" y="179.07" size="1.778" layer="95" rot="R180"/>
+<attribute name="VALUE" x="26.67" y="181.61" size="1.778" layer="96" rot="R180"/>
+</instance>
+<instance part="VO1" gate="G$1" x="76.2" y="238.76" smashed="yes" rot="R270">
+<attribute name="NAME" x="77.47" y="240.03" size="1.778" layer="95" rot="R270"/>
+<attribute name="VALUE" x="74.93" y="237.49" size="1.778" layer="96" rot="R270"/>
+</instance>
+<instance part="VO2" gate="G$1" x="76.2" y="228.6" smashed="yes" rot="R270">
+<attribute name="NAME" x="77.47" y="229.87" size="1.778" layer="95" rot="R270"/>
+<attribute name="VALUE" x="74.93" y="227.33" size="1.778" layer="96" rot="R270"/>
+</instance>
+<instance part="VO3" gate="G$1" x="76.2" y="218.44" smashed="yes" rot="R270">
+<attribute name="NAME" x="77.47" y="219.71" size="1.778" layer="95" rot="R270"/>
+<attribute name="VALUE" x="74.93" y="217.17" size="1.778" layer="96" rot="R270"/>
+</instance>
+<instance part="VO4" gate="G$1" x="76.2" y="208.28" smashed="yes" rot="R270">
+<attribute name="NAME" x="77.47" y="209.55" size="1.778" layer="95" rot="R270"/>
+<attribute name="VALUE" x="74.93" y="207.01" size="1.778" layer="96" rot="R270"/>
+</instance>
+<instance part="VO5" gate="G$1" x="76.2" y="198.12" smashed="yes" rot="R270">
+<attribute name="NAME" x="77.47" y="199.39" size="1.778" layer="95" rot="R270"/>
+<attribute name="VALUE" x="74.93" y="196.85" size="1.778" layer="96" rot="R270"/>
+</instance>
+<instance part="VO6" gate="G$1" x="76.2" y="187.96" smashed="yes" rot="R270">
+<attribute name="NAME" x="77.47" y="189.23" size="1.778" layer="95" rot="R270"/>
+<attribute name="VALUE" x="74.93" y="186.69" size="1.778" layer="96" rot="R270"/>
+</instance>
 <instance part="FRAME1" gate="G$1" x="0" y="0"/>
+<instance part="VIN1" gate="G$1" x="30.48" y="180.34" smashed="yes" rot="R180">
+<attribute name="NAME" x="36.83" y="179.07" size="1.778" layer="95" rot="R180"/>
+<attribute name="VALUE" x="29.21" y="181.61" size="1.778" layer="96" rot="R180"/>
+</instance>
+<instance part="VO7" gate="G$1" x="76.2" y="241.3" smashed="yes" rot="R270">
+<attribute name="NAME" x="80.01" y="242.57" size="1.778" layer="95" rot="R270"/>
+<attribute name="VALUE" x="74.93" y="240.03" size="1.778" layer="96" rot="R270"/>
+</instance>
+<instance part="VO8" gate="G$1" x="76.2" y="231.14" smashed="yes" rot="R270">
+<attribute name="NAME" x="80.01" y="232.41" size="1.778" layer="95" rot="R270"/>
+<attribute name="VALUE" x="74.93" y="229.87" size="1.778" layer="96" rot="R270"/>
+</instance>
+<instance part="VO9" gate="G$1" x="76.2" y="220.98" smashed="yes" rot="R270">
+<attribute name="NAME" x="80.01" y="222.25" size="1.778" layer="95" rot="R270"/>
+<attribute name="VALUE" x="74.93" y="219.71" size="1.778" layer="96" rot="R270"/>
+</instance>
+<instance part="VO10" gate="G$1" x="76.2" y="210.82" smashed="yes" rot="R270">
+<attribute name="NAME" x="80.01" y="212.09" size="1.778" layer="95" rot="R270"/>
+<attribute name="VALUE" x="74.93" y="209.55" size="1.778" layer="96" rot="R270"/>
+</instance>
+<instance part="VO11" gate="G$1" x="76.2" y="200.66" smashed="yes" rot="R270">
+<attribute name="NAME" x="80.01" y="201.93" size="1.778" layer="95" rot="R270"/>
+<attribute name="VALUE" x="74.93" y="199.39" size="1.778" layer="96" rot="R270"/>
+</instance>
+<instance part="VO12" gate="G$1" x="76.2" y="190.5" smashed="yes" rot="R270">
+<attribute name="NAME" x="80.01" y="191.77" size="1.778" layer="95" rot="R270"/>
+<attribute name="VALUE" x="74.93" y="189.23" size="1.778" layer="96" rot="R270"/>
+</instance>
 </instances>
 <busses>
@@
 <segment>
 <pinref part="LED3" gate="G$1" pin="C"/>
-<wire x1="66.04" y1="238.76" x2="73.66" y2="238.76" width="0.1524" layer="91"/>
+<wire x1="66.04" y1="238.76" x2="71.12" y2="238.76" width="0.1524" layer="91"/>
 <pinref part="VO1" gate="G$1" pin="TP"/>
+<pinref part="VO7" gate="G$1" pin="TP"/>
+<wire x1="71.12" y1="238.76" x2="73.66" y2="238.76" width="0.1524" layer="91"/>
+<wire x1="73.66" y1="241.3" x2="71.12" y2="241.3" width="0.1524" layer="91"/>
+<wire x1="71.12" y1="241.3" x2="71.12" y2="238.76" width="0.1524" layer="91"/>
+<junction x="71.12" y="238.76"/>
 </segment>
 </net>
@@
 <segment>
 <pinref part="LED6" gate="G$1" pin="C"/>
-<wire x1="66.04" y1="228.6" x2="73.66" y2="228.6" width="0.1524" layer="91"/>
+<wire x1="66.04" y1="228.6" x2="71.12" y2="228.6" width="0.1524" layer="91"/>
 <pinref part="VO2" gate="G$1" pin="TP"/>
+<pinref part="VO8" gate="G$1" pin="TP"/>
+<wire x1="71.12" y1="228.6" x2="73.66" y2="228.6" width="0.1524" layer="91"/>
+<wire x1="73.66" y1="231.14" x2="71.12" y2="231.14" width="0.1524" layer="91"/>
+<wire x1="71.12" y1="231.14" x2="71.12" y2="228.6" width="0.1524" layer="91"/>
+<junction x="71.12" y="228.6"/>
 </segment>
 </net>
@@
 <segment>
 <pinref part="LED9" gate="G$1" pin="C"/>
-<wire x1="66.04" y1="218.44" x2="73.66" y2="218.44" width="0.1524" layer="91"/>
+<wire x1="66.04" y1="218.44" x2="71.12" y2="218.44" width="0.1524" layer="91"/>
 <pinref part="VO3" gate="G$1" pin="TP"/>
+<pinref part="VO9" gate="G$1" pin="TP"/>
+<wire x1="71.12" y1="218.44" x2="73.66" y2="218.44" width="0.1524" layer="91"/>
+<wire x1="73.66" y1="220.98" x2="71.12" y2="220.98" width="0.1524" layer="91"/>
+<wire x1="71.12" y1="220.98" x2="71.12" y2="218.44" width="0.1524" layer="91"/>
+<junction x="71.12" y="218.44"/>
 </segment>
 </net>
@@
 <segment>
 <pinref part="LED12" gate="G$1" pin="C"/>
-<wire x1="66.04" y1="208.28" x2="73.66" y2="208.28" width="0.1524" layer="91"/>
+<wire x1="66.04" y1="208.28" x2="71.12" y2="208.28" width="0.1524" layer="91"/>
 <pinref part="VO4" gate="G$1" pin="TP"/>
+<pinref part="VO10" gate="G$1" pin="TP"/>
+<wire x1="71.12" y1="208.28" x2="73.66" y2="208.28" width="0.1524" layer="91"/>
+<wire x1="73.66" y1="210.82" x2="71.12" y2="210.82" width="0.1524" layer="91"/>
+<wire x1="71.12" y1="210.82" x2="71.12" y2="208.28" width="0.1524" layer="91"/>
+<junction x="71.12" y="208.28"/>
 </segment>
 </net>
@@
 <segment>
 <pinref part="LED15" gate="G$1" pin="C"/>
-<wire x1="66.04" y1="198.12" x2="73.66" y2="198.12" width="0.1524" layer="91"/>
+<wire x1="66.04" y1="198.12" x2="71.12" y2="198.12" width="0.1524" layer="91"/>
 <pinref part="VO5" gate="G$1" pin="TP"/>
+<pinref part="VO11" gate="G$1" pin="TP"/>
+<wire x1="71.12" y1="198.12" x2="73.66" y2="198.12" width="0.1524" layer="91"/>
+<wire x1="73.66" y1="200.66" x2="71.12" y2="200.66" width="0.1524" layer="91"/>
+<wire x1="71.12" y1="200.66" x2="71.12" y2="198.12" width="0.1524" layer="91"/>
+<junction x="71.12" y="198.12"/>
 </segment>
 </net>
@@
 <segment>
 <pinref part="LED18" gate="G$1" pin="C"/>
-<wire x1="66.04" y1="187.96" x2="73.66" y2="187.96" width="0.1524" layer="91"/>
+<wire x1="66.04" y1="187.96" x2="71.12" y2="187.96" width="0.1524" layer="91"/>
 <pinref part="VO6" gate="G$1" pin="TP"/>
+<pinref part="VO12" gate="G$1" pin="TP"/>
+<wire x1="71.12" y1="187.96" x2="73.66" y2="187.96" width="0.1524" layer="91"/>
+<wire x1="73.66" y1="190.5" x2="71.12" y2="190.5" width="0.1524" layer="91"/>
+<wire x1="71.12" y1="190.5" x2="71.12" y2="187.96" width="0.1524" layer="91"/>
+<junction x="71.12" y="187.96"/>
 </segment>
 </net>
@@
 <wire x1="27.94" y1="208.28" x2="27.94" y2="198.12" width="0.1524" layer="91"/>
 <wire x1="27.94" y1="198.12" x2="27.94" y2="187.96" width="0.1524" layer="91"/>
-<wire x1="27.94" y1="187.96" x2="27.94" y2="182.88" width="0.1524" layer="91"/>
+<wire x1="27.94" y1="187.96" x2="27.94" y2="185.42" width="0.1524" layer="91"/>
 <pinref part="LED16" gate="G$1" pin="A"/>
+<wire x1="27.94" y1="185.42" x2="27.94" y2="182.88" width="0.1524" layer="91"/>
 <wire x1="27.94" y1="187.96" x2="38.1" y2="187.96" width="0.1524" layer="91"/>
 <pinref part="LED13" gate="G$1" pin="A"/>
@@
 <junction x="27.94" y="228.6"/>
 <pinref part="VIN" gate="G$1" pin="TP"/>
-</segment>
-</net>
+<pinref part="VIN1" gate="G$1" pin="TP"/>
+<wire x1="30.48" y1="182.88" x2="30.48" y2="185.42" width="0.1524" layer="91"/>
+<wire x1="30.48" y1="185.42" x2="27.94" y2="185.42" width="0.1524" layer="91"/>
+<junction x="27.94" y="185.42"/>
+</segment>
+</net>

Commit message: final updates before fab.  added new letters for future projects.
Parts:
- added LED19, LED20, LED21, LED22, LED23, LED24: (no value), CyberRailGuru:LED0805
- added VO13, VO14, VO15, VO16: (no value), CyberRailGuru:TEST_POINTPAD1-20
Connections:
- new net N$11: LED24.C, VO16.TP, VO8.TP
- new net N$12: LED21.C, VO15.TP, VO7.TP
- new net N$3: LED19.C, LED20.A
- new net N$4: LED20.C, LED21.A
- new net N$7: LED22.C, LED23.A
- new net N$8: LED23.C, LED24.A
- net VIN: now also LED19.A, LED22.A
- net VOUT1: now also VO9.TP; no longer VO7.TP
- net VOUT2: now also VO10.TP; no longer VO8.TP
- net VOUT3: now also VO11.TP; no longer VO9.TP
- net VOUT4: now also VO12.TP; no longer VO10.TP
- net VOUT5: now also VO13.TP; no longer VO11.TP
- net VOUT6: now also VO14.TP; no longer VO12.TP
Other:
- moved on the sheet: VIN, VIN1, VO10, VO11, VO12, VO7, VO8, VO9
