File: Projects/Power Tower Mast/s/s.brd (EAGLE design)
At the start: 16.5 x 21.6 mm, 37 parts

Commit message: final updates before fab.  added new letters for future projects.
Parts:
- moved LED18 0.16 mm to (8.41, 19.5)
Routing:
- net VIN: track 61.3 -> 53.6 mm, vias 0 -> 6
