File: Projects/Letters Upper 15/m/m.brd (EAGLE design)
At the start: 16.5 x 21.6 mm, 37 parts

Commit message: continued working.
Parts:
- moved VO3 1.91 mm to (5.87, 19.5)
- moved VO11 1.62 mm to (9.21, 17.6)
- moved VO10 1.28 mm to (4.92, 19.5)
- moved VO4 0.95 mm to (10.2, 17.6)
- moved LED9 0.85 mm to (5.08, 17.6), turned to 0 degrees
- moved LED13 0.81 mm to (11.4, 17.8), turned to 0 degrees
- moved LED12 0.50 mm to (9.84, 15.7), turned to 0 degrees
- moved LED10 0.48 mm to (6.67, 15.7), turned to 0 degrees
- moved LED7 0.32 mm to (2.54, 17.0)
- moved LED15 0.32 mm to (14.0, 17.0)
- moved LED11 0.16 mm to (8.26, 13.8), turned to 0 degrees
Routing:
- net N$46: track 1.01 -> 4.66 mm, vias 0 -> 2
- net N$43: track 0.86 -> 3.57 mm
- net VIN: track 46.2 -> 47.7 mm
- net N$48: track 0.86 -> 1.78 mm
- net N$45: track 0.85 -> 1.67 mm
