File: Projects/Letters Upper 15/working/a/a.brd (EAGLE design)
At the start: 16.5 x 21.6 mm, 42 parts

Commit message: continued working.
Parts:
- moved VO8 12.2 mm to (5.87, 13.2)
- moved VO16 12.1 mm to (4.92, 13.0)
- moved VO15 11.9 mm to (9.37, 13.0)
- moved VO7 11.3 mm to (10.3, 13.0)
- moved LED22 8.75 mm to (8.26, 10.8), turned to 0 degrees
- moved LED23 8.72 mm to (6.67, 10.8), turned to 0 degrees
- moved LED24 8.69 mm to (5.08, 10.8), turned to 0 degrees
- moved LED21 8.29 mm to (9.84, 10.8), turned to 0 degrees
- moved LED20 6.58 mm to (11.4, 10.8), turned to 0 degrees
- moved VO6 6.11 mm to (12.9, 3.02)
- moved VO14 5.55 mm to (12.9, 4.60)
- moved LED19 5.40 mm to (14.0, 1.59), turned to 90 degrees
- moved VIN 5.39 mm to (1.43, 0.79)
- moved VO4 5.24 mm to (10.5, 15.4)
- moved VO13 5.15 mm to (12.9, 9.68)
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Routing:
- net VIN: track 0.00 -> 55.9 mm, vias 0 -> 7
- net N$28: track 0.00 -> 11.8 mm, vias 0 -> 2
- net N$20: track 0.00 -> 3.90 mm
- net N$24: track 0.00 -> 3.09 mm
- net N$4: track 0.00 -> 3.09 mm
- net N$7: track 0.00 -> 3.09 mm
- net N$3: track 0.00 -> 3.09 mm
- net N$23: track 0.00 -> 3.09 mm
- net N$19: track 0.00 -> 3.09 mm
- net N$8: track 0.00 -> 3.09 mm
- net N$27: track 0.00 -> 2.79 mm
- net N$2: track 0.00 -> 2.76 mm
- net N$1: track 0.00 -> 2.76 mm
- net VOUT7: track 0.00 -> 2.74 mm
- net N$15: track 0.00 -> 2.25 mm
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