File: Projects/Letters Upper 15/working/b/b.brd (EAGLE design)
At the start: 16.5 x 21.6 mm, 42 parts

Commit message: continued working.
Parts:
- moved VO6 11.6 mm to (4.60, 11.6)
- moved VO14 9.86 mm to (6.19, 11.9)
- moved LED18 8.78 mm to (5.40, 10.8), turned to 0 degrees
- moved LED17 6.51 mm to (7.46, 10.8), turned to 0 degrees
- moved VO5 5.65 mm to (12.2, 11.0)
- moved LED16 4.98 mm to (9.37, 10.8), turned to 0 degrees
- moved LED15 4.67 mm to (11.3, 10.8), turned to 0 degrees
- moved VIN1 4.41 mm to (3.81, 0.79)
- moved VO13 4.06 mm to (12.2, 11.9)
- moved VO4 3.98 mm to (13.3, 16.8)
- moved LED14 3.70 mm to (12.3, 13.4), turned to 270 degrees
- moved VO3 3.34 mm to (6.03, 20.5)
- moved LED13 3.27 mm to (13.5, 15.6), turned to 270 degrees
- moved VO12 3.18 mm to (13.3, 18.6)
- moved VO7 2.91 mm to (12.1, 4.76)
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Routing:
- net VIN: track 0.00 -> 55.6 mm, vias 0 -> 7
- net N$19: track 0.00 -> 5.15 mm
- net N$20: track 0.00 -> 4.26 mm
- net N$11: track 0.00 -> 4.11 mm
- net N$28: track 0.00 -> 4.04 mm
- net N$15: track 0.00 -> 3.73 mm
- net N$2: track 0.00 -> 3.25 mm
- net N$1: track 0.00 -> 3.25 mm
- net N$16: track 0.00 -> 3.09 mm
- net N$7: track 0.00 -> 3.09 mm
- net N$12: track 0.00 -> 3.09 mm
- net N$4: track 0.00 -> 3.09 mm
- net N$3: track 0.00 -> 3.09 mm
- net N$8: track 0.00 -> 3.09 mm
- net N$23: track 0.00 -> 2.95 mm
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