File: Projects/Letters Upper 15/working/h/h.brd (EAGLE design)
At the start: 16.5 x 21.6 mm, 42 parts

Commit message: continued working.
Parts:
- moved LED22 8.86 mm to (7.78, 10.8)
- moved LED23 8.78 mm to (6.35, 10.8)
- moved LED24 8.72 mm to (4.92, 10.8)
- moved LED21 8.60 mm to (9.23, 10.9), turned to 180 degrees
- moved LED20 6.92 mm to (10.7, 10.9), turned to 180 degrees
- moved LED11 6.03 mm to (14.3, 19.4), turned to 270 degrees
- moved LED19 5.09 mm to (13.7, 1.91)
- moved LED18 4.76 mm to (14.0, 4.13)
- moved LED12 4.63 mm to (14.0, 17.0), turned to 270 degrees
- moved LED17 4.45 mm to (14.0, 6.35)
- moved LED10 4.29 mm to (2.22, 19.2), turned to 90 degrees
- moved LED16 4.14 mm to (13.7, 8.57)
- moved LED15 4.13 mm to (14.0, 10.5)
- moved LED14 3.95 mm to (14.1, 12.9), turned to 270 degrees
- moved LED13 3.72 mm to (14.0, 15.3), turned to 270 degrees
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