File: Projects/Letters Upper 15/working/j/j.brd (EAGLE design)
At the start: 16.5 x 21.6 mm, 42 parts

Commit message: continued working.
Parts:
- moved LED19 16.8 mm to (30.8, 7.30)
- moved LED20 15.0 mm to (28.6, 5.87)
- moved LED24 14.6 mm to (20.8, 5.40)
- moved LED22 14.6 mm to (24.3, 5.40)
- moved LED23 14.6 mm to (22.5, 5.40)
- moved LED21 14.5 mm to (26.5, 5.40)
- moved LED7 12.5 mm to (11.1, 5.56)
- moved LED8 12.4 mm to (11.2, 7.58), turned to 90 degrees
- moved LED6 11.7 mm to (10.2, 3.81), turned to 270 degrees
- moved VO3 11.7 mm to (8.73, 8.89)
- moved LED9 11.4 mm to (11.1, 9.47), turned to 90 degrees
- moved VO11 10.8 mm to (8.89, 10.2)
- moved LED18 10.7 mm to (14.6, 19.5), turned to 180 degrees
- moved LED5 10.3 mm to (8.41, 2.38), turned to 0 degrees
- moved VO16 9.86 mm to (14.3, 3.49)
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