File: Projects/Letters Upper 15/working/k/k.brd (EAGLE design)
At the start: 16.5 x 21.6 mm, 42 parts

Commit message: continued working.
Parts:
- moved LED11 9.79 mm to (4.92, 10.2)
- moved LED12 7.88 mm to (6.35, 12.4)
- moved LED17 7.24 mm to (6.99, 8.89), turned to 0 degrees
- moved LED16 6.36 mm to (13.7, 19.1), turned to 0 degrees
- moved LED13 6.32 mm to (8.26, 13.7), turned to 0 degrees
- moved LED18 5.54 mm to (8.57, 7.62), turned to 0 degrees
- moved LED14 4.02 mm to (9.84, 15.6), turned to 0 degrees
- moved LED19 4.02 mm to (10.2, 5.71), turned to 0 degrees
- moved LED10 4.00 mm to (2.54, 19.8), turned to 90 degrees
- moved LED15 3.62 mm to (11.7, 17.5), turned to 0 degrees
- moved LED1 2.00 mm to (2.46, 2.04), turned to 90 degrees
- moved LED9 1.93 mm to (2.44, 18.0), turned to 90 degrees
- moved LED21 1.87 mm to (14.0, 2.26), turned to 0 degrees
- moved LED20 1.77 mm to (12.1, 3.81), turned to 0 degrees
- moved LED3 0.95 mm to (2.54, 6.03)
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