File: Projects/Letters Upper 15/j/j.sch (EAGLE design)
At the start: 42 parts

Commit message: 
Parts:
- removed LED19, LED20, LED21, LED22, LED23, LED24: (no value), CyberRailGuru:LED0805
- removed VO13, VO14, VO15, VO16: (no value), CyberRailGuru:TEST_POINTPAD1-20
Connections:
- removed net N$1: LED22.C, LED23.A
- removed net N$2: LED23.C, LED24.A
- removed net N$27: LED20.C, LED21.A
- removed net N$28: LED19.C, LED20.A
- removed net N$5: LED24.C, VO16.TP, VO8.TP
- removed net VOUT7: LED21.C, VO15.TP, VO7.TP
- net VIN: no longer LED19.A, LED22.A
- net VOUT1: now also VO7.TP; no longer VO9.TP
- net VOUT2: now also VO8.TP; no longer VO10.TP
- net VOUT3: now also VO9.TP; no longer VO11.TP
- net VOUT4: now also VO10.TP; no longer VO12.TP
- net VOUT5: now also VO11.TP; no longer VO13.TP
- net VOUT6: now also VO12.TP; no longer VO14.TP
Other:
- moved on the sheet: VO10, VO11, VO12, VO7, VO8, VO9
